File: PCB/Rev .6/IDE_Bridge.kicad_pcb (KiCad board)
At the start: 2 copper layers, 48 x 52 mm, 95 parts, among them J1 IDE Connector, P1 USB_C_Plug_USB2.0, SW1 BOOTSEL, U1 74HCT245, U2 74HCT125, U3 74HCT125, U4 74HCT245, U5 RP2354B, U6 TVS, U7 LDO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

Commit message: Add files via upload
Routing:
- net GND: vias 37 -> 38
Changed lines of the file:
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@@
+	)
+	(via
+		(at 156.21 97.74)
+		(size 0.6)
+		(drill 0.3)
+		(layers "F.Cu" "B.Cu")
+		(free yes)
+		(net 6)
 	)
 	(via
